File: Design Files/Strelka_Flight_Computer/Actuators.kicad_sch (KiCad schematic)
At the start: 10 parts, among them J3 DB125-3.5-4P-GN-S, J4 SM06B-GHS-TB(LF)(SN)

Commit message: First go at routing
Connections:
- net Ematch_Drogue1/EMATCH+: now also J3.4 (Pin_4)
- net Ematch_Drogue1/EMATCH-: now also J3.3 (Pin_3)
- net Ematch_Main/EMATCH-: now also J3.1 (Pin_1)
Changed lines of the file:
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@@
   (junction (at 168.91 85.09) (diameter 0) (color 0 0 0 0)
   )
-  (wire (pts (xy 91.44 81.28) (xy 99.06 81.28))
+  (wire (pts (xy 91.44 81.915) (xy 99.06 81.915))
     (stroke (width 0) (type default) (color 0 0 0 0))
   )
@@
     (stroke (width 0) (type default) (color 0 0 0 0))
   )
-  (wire (pts (xy 101.6 63.5) (xy 101.6 69.85))
+  (wire (pts (xy 101.6 62.865) (xy 101.6 69.85))
     (stroke (width 0) (type default) (color 0 0 0 0))
   )
@@
     (stroke (width 0) (type default) (color 0 0 0 0))
   )
-  (wire (pts (xy 91.44 46.99) (xy 101.6 46.99))
+  (wire (pts (xy 91.44 46.355) (xy 101.6 46.355))
     (stroke (width 0) (type default) (color 0 0 0 0))
   )
@@
     (stroke (width 0) (type default) (color 0 0 0 0))
   )
-  (wire (pts (xy 91.44 63.5) (xy 101.6 63.5))
+  (wire (pts (xy 91.44 62.865) (xy 101.6 62.865))
     (stroke (width 0) (type default) (color 0 0 0 0))
   )
@@
     (stroke (width 0) (type default) (color 0 0 0 0))
   )
-  (wire (pts (xy 99.06 74.93) (xy 99.06 81.28))
+  (wire (pts (xy 99.06 74.93) (xy 99.06 81.915))
     (stroke (width 0) (type default) (color 0 0 0 0))
   )
@@
     (effects (font (size 1.27 1.27)) (justify right))
   )
-  (hierarchical_label "MAIN_L" (shape input) (at 101.6 46.99 0)
+  (hierarchical_label "MAIN_L" (shape input) (at 101.6 46.355 0)
     (effects (font (size 1.27 1.27)) (justify left))
   )
@@
       (effects (font (size 1.27 1.27)) (justify left top))
     )
-    (pin "CONT_TEST" input (at 65.786 78.74 90)
-      (effects (font (size 1.27 1.27)) (justify right))
-    )
-    (pin "EMATCH_Cont" input (at 91.44 115.824 0)
-      (effects (font (size 1.27 1.27)) (justify right))
-    )
-    (pin "EMATCH+" input (at 91.44 83.566 0)
-      (effects (font (size 1.27 1.27)) (justify right))
-    )
-    (pin "EMATCH-" input (at 91.44 81.788 0)
-      (effects (font (size 1.27 1.27)) (justify right))
-    )
-    (pin "FIRE_L" input (at 91.44 101.092 0)
-      (effects (font (size 1.27 1.27)) (justify right))
-    )
-    (pin "FIRE_H" input (at 91.44 103.124 0)
+    (pin "CONT_TEST" input (at 64.77 78.74 90)
+      (effects (font (size 1.27 1.27)) (justify right))
+    )
+    (pin "EMATCH_Cont" input (at 91.44 115.57 0)
+      (effects (font (size 1.27 1.27)) (justify right))
+    )
+    (pin "EMATCH+" input (at 91.44 83.82 0)
+      (effects (font (size 1.27 1.27)) (justify right))
+    )
+    (pin "EMATCH-" input (at 91.44 81.915 0)
+      (effects (font (size 1.27 1.27)) (justify right))
+    )
+    (pin "FIRE_L" input (at 91.44 100.33 0)
+      (effects (font (size 1.27 1.27)) (justify right))
+    )
+    (pin "FIRE_H" input (at 91.44 102.87 0)
       (effects (font (size 1.27 1.27)) (justify right))
     )
@@
       (effects (font (size 1.27 1.27)) (justify left top))
     )
-    (pin "CONT_TEST" input (at 65.786 67.31 270)
-      (effects (font (size 1.27 1.27)) (justify left))
-    )
-    (pin "EMATCH_Cont" input (at 91.44 38.354 0)
+    (pin "CONT_TEST" input (at 64.77 67.31 270)
+      (effects (font (size 1.27 1.27)) (justify left))
+    )
+    (pin "EMATCH_Cont" input (at 91.44 38.1 0)
       (effects (font (size 1.27 1.27)) (justify right))
     )
@@
       (effects (font (size 1.27 1.27)) (justify right))
     )
-    (pin "EMATCH-" input (at 91.44 62.992 0)
-      (effects (font (size 1.27 1.27)) (justify right))
-    )
-    (pin "FIRE_L" input (at 91.44 46.482 0)
-      (effects (font (size 1.27 1.27)) (justify right))
-    )
-    (pin "FIRE_H" input (at 91.44 48.514 0)
-      (effects (font (size 1.27 1.27)) (justify right))
-    )
+    (pin "EMATCH-" input (at 91.44 62.865 0)
+      (effects (font (size 1.27 1.27)) (justify right))
+    )
+    (pin "FIRE_L" input (at 91.44 46.355 0)
+      (effects (font (size 1.27 1.27)) (justify right))
+    )
+    (pin "FIRE_H" input (at 91.44 48.26 0)
+      (effects (font (size 1.27 1.27)) (justify right))
+    )

Commit message: Creating BOM
Parts:
- J4: LCSC# (none) -> C133065; MANUFACTURER JST -> (none); MAXIMUM_PACKAGE_HEIGHT 4.25mm -> (none); PARTREV N/A -> (none); STANDARD Manufacturer Recommendations -> (none)
Changed lines of the file:
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@@
       (effects (font (size 1.27 1.27)) (justify left bottom) hide)
     )
-    (property "PARTREV" "N/A" (id 4) (at 236.22 92.71 0)
+    (property "LCSC#" "C133065" (id 4) (at 236.22 92.71 0)
       (effects (font (size 1.27 1.27)) (justify left bottom) hide)
     )
-    (property "STANDARD" "Manufacturer Recommendations" (id 5) (at 236.22 92.71 0)
-      (effects (font (size 1.27 1.27)) (justify left bottom) hide)
-    )
-    (property "MAXIMUM_PACKAGE_HEIGHT" "4.25mm" (id 6) (at 236.22 92.71 0)
-      (effects (font (size 1.27 1.27)) (justify left bottom) hide)
-    )
-    (property "MANUFACTURER" "JST" (id 7) (at 236.22 92.71 0)
-      (effects (font (size 1.27 1.27)) (justify left bottom) hide)
-    )
