File: Design Files/Strelka_Flight_Computer/Strelka_Flight_Computer.kicad_sch (KiCad schematic)
At the start: 10 parts

Commit message: PCB ordered
Connections:
- no-connect marks 5 -> 3
Other:
- removed sheet Status_Output
- sheet Data_Interfaces ports: added none; removed RX_PAD, TX_PAD
- sheet Power ports: added none; removed BOOST_EN
- sheet STM32F405 ports: added GPIO_PA10, GPIO_PA9; removed USART1_RX, USART1_TX
