File: Design Files/Strelka_Flight_Computer/Data_Interfaces.kicad_sch (KiCad schematic)
At the start: 5 parts, among them J2 SM04B-GHS-TB(LF)(SN)-, J6 USB_B_Micro, U8 USBLC6-2SC6

Commit message: PCB ordered
Parts:
- removed TP1, TP2: TestPoint, TestPoint:TestPoint_Pad_2.0x2.0mm, symbol Connector:TestPoint
Changed lines of the file:
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@@
 (kicad_sch (version 20211123) (generator eeschema)
   (paper "A4")
+  (junction (at 212.725 41.91) (diameter 0) (color 0 0 0 0)
+  )
   (junction (at 177.165 62.23) (diameter 0) (color 0 0 0 0)
   )
@@
     (stroke (width 0) (type default) (color 0 0 0 0))
   )
-  (wire (pts (xy 212.725 41.91) (xy 184.785 41.91))
+  (wire (pts (xy 184.785 41.91) (xy 212.725 41.91))
     (stroke (width 0) (type default) (color 0 0 0 0))
   )
@@
     (stroke (width 0) (type default) (color 0 0 0 0))
   )
-  (wire (pts (xy 198.755 79.375) (xy 210.82 79.375))
-    (stroke (width 0) (type default) (color 0 0 0 0))
-  )
   (wire (pts (xy 205.105 44.45) (xy 216.535 44.45))
     (stroke (width 0) (type default) (color 0 0 0 0))
@@
   )
   (wire (pts (xy 174.625 62.23) (xy 177.165 62.23))
-    (stroke (width 0) (type default) (color 0 0 0 0))
-  )
-  (wire (pts (xy 189.23 83.185) (xy 210.82 83.185))
     (stroke (width 0) (type default) (color 0 0 0 0))
   )
@@
     (effects (font (size 1.27 1.27)) (justify left))
   )
-  (hierarchical_label "TX_PAD" (shape input) (at 210.82 79.375 0)
-    (effects (font (size 1.27 1.27)) (justify left))
-  )
-  (hierarchical_label "RX_PAD" (shape input) (at 210.82 83.185 0)
-    (effects (font (size 1.27 1.27)) (justify left))
-  )
   (hierarchical_label "USB_D+" (shape input) (at 216.535 44.45 0)
     (effects (font (size 1.27 1.27)) (justify left))
   )
-  (symbol (lib_id "Connector:TestPoint") (at 198.755 79.375 0) (unit 1)
-    (in_bom yes) (on_board yes) (fields_autoplaced)
-    (property "Reference" "TP2" (id 0) (at 200.66 74.8029 0)
-      (effects (font (size 1.27 1.27)) (justify left))
-    )
-    (property "Value" "TestPoint" (id 1) (at 200.66 77.3429 0)
-      (effects (font (size 1.27 1.27)) (justify left))
-    )
-    (property "Footprint" "TestPoint:TestPoint_Pad_2.0x2.0mm" (id 2) (at 203.835 79.375 0)
-      (effects (font (size 1.27 1.27)) hide)
-    )
-    (property "Datasheet" "~" (id 3) (at 203.835 79.375 0)
+  (symbol (lib_id "power:PWR_FLAG") (at 212.725 41.91 0) (unit 1)
+    (in_bom yes) (on_board yes) (fields_autoplaced)
+    (property "Reference" "#FLG0109" (id 0) (at 212.725 40.005 0)
+      (effects (font (size 1.27 1.27)) hide)
+    )
+    (property "Value" "PWR_FLAG" (id 1) (at 212.725 36.83 0))
+    (property "Footprint" "" (id 2) (at 212.725 41.91 0)
+      (effects (font (size 1.27 1.27)) hide)
+    )
+    (property "Datasheet" "~" (id 3) (at 212.725 41.91 0)
       (effects (font (size 1.27 1.27)) hide)
     )
@@
       (effects (font (size 1.27 1.27)) hide)
     )
-    (pin "1")
-  )
-  (symbol (lib_id "Connector:TestPoint") (at 189.23 83.185 0) (unit 1)
-    (in_bom yes) (on_board yes) (fields_autoplaced)
-    (property "Reference" "TP1" (id 0) (at 191.135 78.6129 0)
-      (effects (font (size 1.27 1.27)) (justify left))
-    )
-    (property "Value" "TestPoint" (id 1) (at 191.135 81.1529 0)
-      (effects (font (size 1.27 1.27)) (justify left))
-    )
-    (property "Footprint" "TestPoint:TestPoint_Pad_2.0x2.0mm" (id 2) (at 194.31 83.185 0)
-      (effects (font (size 1.27 1.27)) hide)
-    )
-    (property "Datasheet" "~" (id 3) (at 194.31 83.185 0)
-      (effects (font (size 1.27 1.27)) hide)
-    )
