File: Design Files/Strelka_Flight_Computer/Power.kicad_sch (KiCad schematic)
At the start: 41 parts, among them J1 1S_LiPo_LARGE_HOLE_XT-30, Q1 CJK2333, Q2 CJK2333, SW3 SM02B-GHS-TB(LF)(SN), U16 TPS61085DGKR, U2 AP9101CK6, U3 AMS1117-3.3

Commit message: redo placement
Parts:
- C41: footprint Capacitor_THT:C_Radial_D8.0mm_H11.5mm_P3.50mm -> Footprints:ULR158M0JF1ARR
- C55: footprint Capacitor_SMD:C_0603_1608Metric -> Capacitor_SMD:C_0805_2012Metric
Connections:
- net GND: now also U16.4 (PGND)
- net VDC: now also U16.7 (FREQ)
- net at R62.1, R63.2: now also U16.2 (FB)
- net at R61.2: now also U16.1 (COMP)
- net at U16.5 (SW): now also D14.2 (A), L2.2
Changed lines of the file:
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@@
     (stroke (width 0) (type default) (color 0 0 0 0))
   )
-  (wire (pts (xy 110.49 143.51) (xy 105.41 143.51))
+  (wire (pts (xy 104.775 143.51) (xy 110.49 143.51))
     (stroke (width 0) (type default) (color 0 0 0 0))
   )
@@
     (stroke (width 0) (type default) (color 0 0 0 0))
   )
+  (wire (pts (xy 104.775 151.765) (xy 105.41 151.765))
+    (stroke (width 0) (type default) (color 0 0 0 0))
+  )
   (wire (pts (xy 83.82 74.93) (xy 91.44 74.93))
     (stroke (width 0) (type default) (color 0 0 0 0))
@@
     (stroke (width 0) (type solid) (color 0 0 0 0))
   )
-  (wire (pts (xy 80.01 149.86) (xy 74.93 149.86))
+  (wire (pts (xy 80.01 149.225) (xy 74.93 149.225))
     (stroke (width 0) (type default) (color 0 0 0 0))
   )
@@
     (stroke (width 0) (type default) (color 0 0 0 0))
   )
-  (wire (pts (xy 105.41 149.86) (xy 113.03 149.86))
+  (wire (pts (xy 104.775 149.225) (xy 113.03 149.225))
     (stroke (width 0) (type default) (color 0 0 0 0))
   )
@@
     (stroke (width 0) (type default) (color 0 0 0 0))
   )
-  (wire (pts (xy 115.57 146.05) (xy 105.41 146.05))
+  (wire (pts (xy 104.775 146.05) (xy 115.57 146.05))
     (stroke (width 0) (type default) (color 0 0 0 0))
   )
@@
     (stroke (width 0) (type default) (color 0 0 0 0))
   )
-  (wire (pts (xy 74.93 149.86) (xy 74.93 143.51))
+  (wire (pts (xy 74.93 149.225) (xy 74.93 143.51))
     (stroke (width 0) (type default) (color 0 0 0 0))
   )
@@
     (stroke (width 0) (type default) (color 0 0 0 0))
   )
+  (wire (pts (xy 105.41 151.765) (xy 105.41 163.83))
+    (stroke (width 0) (type default) (color 0 0 0 0))
+  )
   (wire (pts (xy 74.93 143.51) (xy 77.47 143.51))
     (stroke (width 0) (type default) (color 0 0 0 0))
   )
-  (wire (pts (xy 105.41 152.4) (xy 105.41 163.83))
-    (stroke (width 0) (type default) (color 0 0 0 0))
-  )
   (wire (pts (xy 80.01 152.4) (xy 80.01 158.75))
     (stroke (width 0) (type default) (color 0 0 0 0))
   )
-  (wire (pts (xy 113.03 149.86) (xy 113.03 152.4))
+  (wire (pts (xy 113.03 149.225) (xy 113.03 152.4))
     (stroke (width 0) (type default) (color 0 0 0 0))
   )
@@
       (effects (font (size 1.27 1.27)) (justify left))
     )
-    (property "Footprint" "Capacitor_SMD:C_0603_1608Metric" (id 2) (at 139.7 149.86 0)
+    (property "Footprint" "Capacitor_SMD:C_0805_2012Metric" (id 2) (at 139.7 149.86 0)
       (effects (font (size 1.27 1.27)) hide)
     )
@@
       (effects (font (size 1.27 1.27)) (justify left))
     )
-    (property "Footprint" "Capacitor_THT:C_Radial_D8.0mm_H11.5mm_P3.50mm" (id 2) (at 101.6 54.61 0)
-      (effects (font (size 1.27 1.27)) hide)
-    )
+    (property "Footprint" "Footprints:ULR158M0JF1ARR" (id 2) (at 101.6 54.61 0)
+      (effects (font (size 1.27 1.27)) hide)
+    )

Commit message: PCB ordered
Parts:
- added TP1, TP3, TP4: TestPoint, TestPoint:TestPoint_Pad_1.0x1.0mm, symbol Connector:TestPoint
Connections:
- net +3V3: now also TP4.1
- net +5VA: now also TP3.1
- net VDC: now also TP1.1
Changed lines of the file:
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@@
   (junction (at 66.04 143.51) (diameter 0) (color 0 0 0 0)
   )
+  (junction (at 83.82 68.58) (diameter 0) (color 0 0 0 0)
+  )
   (junction (at 171.45 74.93) (diameter 1.016) (color 0 0 0 0)
   )
@@
   (junction (at 148.59 163.83) (diameter 0) (color 0 0 0 0)
   )
+  (junction (at 131.445 143.51) (diameter 0) (color 0 0 0 0)
+  )
   (junction (at 129.54 163.83) (diameter 0) (color 0 0 0 0)
   )
@@
   )
   (junction (at 214.63 139.7) (diameter 0) (color 0 0 0 0)
+  )
+  (junction (at 217.17 35.56) (diameter 0) (color 0 0 0 0)
   )
   (junction (at 80.01 143.51) (diameter 0) (color 0 0 0 0)
@@
     (stroke (width 0) (type default) (color 0 0 0 0))
   )
+  (wire (pts (xy 77.47 68.58) (xy 83.82 68.58))
+    (stroke (width 0) (type default) (color 0 0 0 0))
+  )
   (wire (pts (xy 128.27 118.11) (xy 121.92 118.11))
     (stroke (width 0) (type default) (color 0 0 0 0))
@@
     (stroke (width 0) (type default) (color 0 0 0 0))
   )
+  (wire (pts (xy 131.445 143.51) (xy 139.7 143.51))
+    (stroke (width 0) (type default) (color 0 0 0 0))
+  )
   (polyline (pts (xy 25.4 109.22) (xy 162.56 109.22))
     (stroke (width 0) (type default) (color 0 0 0 0))
@@
     (stroke (width 0) (type default) (color 0 0 0 0))
   )
+  (wire (pts (xy 77.47 67.31) (xy 77.47 68.58))
+    (stroke (width 0) (type default) (color 0 0 0 0))
+  )
   (wire (pts (xy 101.6 124.46) (xy 109.22 124.46))
     (stroke (width 0) (type default) (color 0 0 0 0))
@@
     (stroke (width 0) (type default) (color 0 0 0 0))
   )
-  (wire (pts (xy 129.54 143.51) (xy 139.7 143.51))
+  (wire (pts (xy 129.54 143.51) (xy 131.445 143.51))
     (stroke (width 0) (type default) (color 0 0 0 0))
   )
@@
     (effects (font (size 1.27 1.27)) (justify left bottom))
   )
-  (text "Vin = 4.2-2.5V\nVo = 3.29-1.96V" (at 87.63 72.39 0)
+  (text "Vin = 4.2-2.5V\nVo = 3.29-1.96V" (at 86.995 69.215 0)
     (effects (font (size 1.27 1.27)) (justify left bottom))
   )
@@
     (pin "2")
   )
+  (symbol (lib_id "Connector:TestPoint") (at 217.17 35.56 0) (unit 1)
+    (in_bom yes) (on_board yes) (fields_autoplaced)
+    (property "Reference" "TP4" (id 0) (at 219.71 30.9879 0)
+      (effects (font (size 1.27 1.27)) (justify left))
+    )
+    (property "Value" "TestPoint" (id 1) (at 219.71 33.5279 0)
+      (effects (font (size 1.27 1.27)) (justify left))
+    )
+    (property "Footprint" "TestPoint:TestPoint_Pad_1.0x1.0mm" (id 2) (at 222.25 35.56 0)
+      (effects (font (size 1.27 1.27)) hide)
+    )
+    (property "Datasheet" "~" (id 3) (at 222.25 35.56 0)
+      (effects (font (size 1.27 1.27)) hide)
+    )
+    (pin "1")
+  )
   (symbol (lib_id "Switch:SW_DIP_x01") (at 92.71 48.26 0) (unit 1)
     (in_bom yes) (on_board yes) (fields_autoplaced)
@@
     (pin "1")
     (pin "2")
+  )
+  (symbol (lib_id "Connector:TestPoint") (at 139.7 143.51 0) (unit 1)
+    (in_bom yes) (on_board yes) (fields_autoplaced)
+    (property "Reference" "TP3" (id 0) (at 142.24 138.9379 0)
+      (effects (font (size 1.27 1.27)) (justify left))
+    )
+    (property "Value" "TestPoint" (id 1) (at 142.24 141.4779 0)
+      (effects (font (size 1.27 1.27)) (justify left))
+    )
+    (property "Footprint" "TestPoint:TestPoint_Pad_1.0x1.0mm" (id 2) (at 144.78 143.51 0)
+      (effects (font (size 1.27 1.27)) hide)
+    )
+    (property "Datasheet" "~" (id 3) (at 144.78 143.51 0)
+      (effects (font (size 1.27 1.27)) hide)
+    )
+    (pin "1")
   )
   (symbol (lib_id "TPS61085DGKR:TPS61085DGKR") (at 97.79 140.335 0) (unit 1)
@@
     (pin "1")
   )
+  (symbol (lib_id "Connector:TestPoint") (at 55.88 143.51 0) (unit 1)
+    (in_bom yes) (on_board yes) (fields_autoplaced)
+    (property "Reference" "TP1" (id 0) (at 58.42 138.9379 0)
+      (effects (font (size 1.27 1.27)) (justify left))
+    )
+    (property "Value" "TestPoint" (id 1) (at 58.42 141.4779 0)
+      (effects (font (size 1.27 1.27)) (justify left))
+    )
+    (property "Footprint" "TestPoint:TestPoint_Pad_1.0x1.0mm" (id 2) (at 60.96 143.51 0)
+      (effects (font (size 1.27 1.27)) hide)
+    )
+    (property "Datasheet" "~" (id 3) (at 60.96 143.51 0)
+      (effects (font (size 1.27 1.27)) hide)
+    )
+    (pin "1")
+  )
   (symbol (lib_id "Device:L_Small") (at 91.44 133.35 90) (unit 1)
     (in_bom yes) (on_board yes)
@@
     (pin "2")
   )
+  (symbol (lib_id "power:PWR_FLAG") (at 77.47 67.31 0) (unit 1)
+    (in_bom yes) (on_board yes) (fields_autoplaced)
+    (property "Reference" "#FLG0111" (id 0) (at 77.47 65.405 0)
+      (effects (font (size 1.27 1.27)) hide)
+    )
+    (property "Value" "PWR_FLAG" (id 1) (at 77.47 62.23 0))
+    (property "Footprint" "" (id 2) (at 77.47 67.31 0)
+      (effects (font (size 1.27 1.27)) hide)
+    )
+    (property "Datasheet" "~" (id 3) (at 77.47 67.31 0)
+      (effects (font (size 1.27 1.27)) hide)
+    )
+    (pin "1")
+  )
   (symbol (lib_id "power:GND") (at 213.36 43.18 0) (unit 1)
     (in_bom yes) (on_board yes) (fields_autoplaced)
@@
     (pin "2")
   )
+  (symbol (lib_id "power:PWR_FLAG") (at 131.445 143.51 0) (unit 1)
+    (in_bom yes) (on_board yes) (fields_autoplaced)
+    (property "Reference" "#FLG0110" (id 0) (at 131.445 141.605 0)
+      (effects (font (size 1.27 1.27)) hide)
+    )
+    (property "Value" "PWR_FLAG" (id 1) (at 131.445 138.43 0))
+    (property "Footprint" "" (id 2) (at 131.445 143.51 0)
+      (effects (font (size 1.27 1.27)) hide)
+    )
+    (property "Datasheet" "~" (id 3) (at 131.445 143.51 0)
+      (effects (font (size 1.27 1.27)) hide)
+    )
+    (pin "1")
+  )
   (symbol (lib_id "Device:C_Small") (at 115.57 120.65 0) (unit 1)
