File: Design Files/Strelka_Flight_Computer/STM32F405.kicad_sch (KiCad schematic)
At the start: 30 parts, among them SW1 SW_Push, SW2 SW_Push, U5 STM32F405RGTx, Y1 Q13FC1350000200, Y2 X322524MOB4SI

Commit message: redo placement
Parts:
- SW1, SW2: footprint Button_Switch_SMD:SW_Push_1P1T_NO_CK_KSC6xxJ -> Button_Switch_SMD:SW_Push_SPST_NO_Alps_SKRK
Changed lines of the file:
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@@
+    (stroke (width 0) (type default) (color 0 0 0 0))
+  )
+  (wire (pts (xy 85.09 76.2) (xy 87.63 76.2))
+    (stroke (width 0) (type default) (color 0 0 0 0))
+  )
+  (wire (pts (xy 87.63 85.09) (xy 87.63 87.63))
+    (stroke (width 0) (type default) (color 0 0 0 0))
+  )
+  (wire (pts (xy 119.38 49.53) (xy 129.54 49.53))
+    (stroke (width 0) (type default) (color 0 0 0 0))
+  )
+  (wire (pts (xy 111.76 125.73) (xy 118.11 125.73))
+    (stroke (width 0) (type default) (color 0 0 0 0))
+  )
+  (wire (pts (xy 217.17 147.32) (xy 229.87 147.32))
+    (stroke (width 0) (type default) (color 0 0 0 0))
+  )
+  (polyline (pts (xy 223.52 49.53) (xy 266.7 49.53))
+    (stroke (width 0) (type default) (color 0 0 0 0))
+  )
+  (polyline (pts (xy 223.52 49.53) (xy 223.52 71.12))
+    (stroke (width 0) (type default) (color 0 0 0 0))
+  )
+  (wire (pts (xy 110.49 80.01) (xy 110.49 81.28))
     (stroke (width 0) (type default) (color 0 0 0 0))
   )
@@
     (stroke (width 0) (type default) (color 0 0 0 0))
   )
-  (wire (pts (xy 87.63 85.09) (xy 87.63 87.63))
-    (stroke (width 0) (type default) (color 0 0 0 0))
-  )
-  (wire (pts (xy 119.38 49.53) (xy 129.54 49.53))
-    (stroke (width 0) (type default) (color 0 0 0 0))
-  )
-  (wire (pts (xy 111.76 125.73) (xy 118.11 125.73))
-    (stroke (width 0) (type default) (color 0 0 0 0))
-  )
-  (wire (pts (xy 217.17 147.32) (xy 229.87 147.32))
-    (stroke (width 0) (type default) (color 0 0 0 0))
-  )
-  (polyline (pts (xy 223.52 49.53) (xy 266.7 49.53))
-    (stroke (width 0) (type default) (color 0 0 0 0))
-  )
-  (polyline (pts (xy 223.52 49.53) (xy 223.52 71.12))
-    (stroke (width 0) (type default) (color 0 0 0 0))
-  )
-  (wire (pts (xy 110.49 80.01) (xy 110.49 81.28))
-    (stroke (width 0) (type default) (color 0 0 0 0))
-  )
   (polyline (pts (xy 222.25 49.53) (xy 222.25 71.12))
+    (stroke (width 0) (type default) (color 0 0 0 0))
+  )
+  (wire (pts (xy 73.66 76.2) (xy 74.93 76.2))
     (stroke (width 0) (type default) (color 0 0 0 0))
   )
@@
   )
   (wire (pts (xy 217.17 144.78) (xy 222.25 144.78))
-    (stroke (width 0) (type default) (color 0 0 0 0))
-  )
-  (wire (pts (xy 73.66 76.2) (xy 77.47 76.2))
     (stroke (width 0) (type default) (color 0 0 0 0))
   )
@@
     (property "Reference" "SW2" (id 0) (at 88.9 51.181 0))
     (property "Value" "SW_Push" (id 1) (at 88.9 53.4924 0))
-    (property "Footprint" "Button_Switch_SMD:SW_Push_1P1T_NO_CK_KSC6xxJ" (id 2) (at 88.9 53.34 0)
+    (property "Footprint" "Button_Switch_SMD:SW_Push_SPST_NO_Alps_SKRK" (id 2) (at 88.9 53.34 0)
       (effects (font (size 1.27 1.27)) hide)
     )
@@
     )
     (property "Datasheet" "~" (id 3) (at 185.42 142.24 0)
+      (effects (font (size 1.27 1.27)) hide)
+    )
+    (pin "1")
+    (pin "2")
+  )
+  (symbol (lib_id "Nebula-rescue:SW_Push-Switch-H7_FlightComputer-rescue") (at 80.01 76.2 0) (unit 1)
+    (in_bom yes) (on_board yes)
+    (property "Reference" "SW1" (id 0) (at 80.01 68.961 0))
+    (property "Value" "SW_Push" (id 1) (at 80.01 71.2724 0))
+    (property "Footprint" "Button_Switch_SMD:SW_Push_SPST_NO_Alps_SKRK" (id 2) (at 80.01 71.12 0)
+      (effects (font (size 1.27 1.27)) hide)
+    )
+    (property "Datasheet" "~" (id 3) (at 80.01 71.12 0)
       (effects (font (size 1.27 1.27)) hide)
     )
@@
       (effects (font (size 1.27 1.27)) hide)
     )
-    (pin "1")
-    (pin "2")
-  )
-  (symbol (lib_id "Nebula-rescue:SW_Push-Switch-H7_FlightComputer-rescue") (at 82.55 76.2 0) (unit 1)
-    (in_bom yes) (on_board yes)
-    (property "Reference" "SW1" (id 0) (at 82.55 68.961 0))
-    (property "Value" "SW_Push" (id 1) (at 82.55 71.2724 0))
-    (property "Footprint" "Button_Switch_SMD:SW_Push_1P1T_NO_CK_KSC6xxJ" (id 2) (at 82.55 71.12 0)
-      (effects (font (size 1.27 1.27)) hide)
-    )
-    (property "Datasheet" "~" (id 3) (at 82.55 71.12 0)
-      (effects (font (size 1.27 1.27)) hide)
-    )

Commit message: PCB ordered
Connections:
- net USART1_RX renamed GPIO_PA10
- net USART1_TX renamed GPIO_PA9
Changed lines of the file:
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@@
   (junction (at 137.16 59.69) (diameter 0) (color 0 0 0 0)
   )
+  (junction (at 130.81 59.69) (diameter 0) (color 0 0 0 0)
+  )
   (junction (at 119.38 49.53) (diameter 0) (color 0 0 0 0)
   )
@@
   )
   (junction (at 149.86 46.99) (diameter 0) (color 0 0 0 0)
+  )
+  (junction (at 143.51 35.56) (diameter 0) (color 0 0 0 0)
   )
   (junction (at 162.56 46.99) (diameter 0) (color 0 0 0 0)
@@
     (effects (font (size 1.27 1.27)) (justify right))
   )
-  (hierarchical_label "USART1_TX" (shape input) (at 160.02 90.17 0)
+  (hierarchical_label "GPIO_PA9" (shape input) (at 160.02 90.17 0)
     (effects (font (size 1.27 1.27)) (justify left))
   )
@@
     (effects (font (size 1.27 1.27)) (justify right))
   )
-  (hierarchical_label "USART1_RX" (shape input) (at 160.02 92.71 0)
+  (hierarchical_label "GPIO_PA10" (shape input) (at 160.02 92.71 0)
     (effects (font (size 1.27 1.27)) (justify left))
   )
@@
   )
   (symbol (lib_id "Device:FerriteBead_Small") (at 155.448 35.56 270) (mirror x) (unit 1)
-    (in_bom yes) (on_board yes) (fields_autoplaced)
-    (property "Reference" "FB1" (id 0) (at 155.4861 28.575 90))
-    (property "Value" "BLM18PG221SN1D" (id 1) (at 155.4861 31.115 90))
+    (in_bom yes) (on_board yes)
+    (property "Reference" "FB1" (id 0) (at 155.575 30.48 90))
+    (property "Value" "BLM18PG221SN1D" (id 1) (at 155.575 32.385 90))
     (property "Footprint" "Inductor_SMD:L_0603_1608Metric" (id 2) (at 155.448 37.338 90)
       (effects (font (size 1.27 1.27)) hide)
@@
     (pin "2")
   )
+  (symbol (lib_id "power:PWR_FLAG") (at 143.51 35.56 0) (unit 1)
+    (in_bom yes) (on_board yes) (fields_autoplaced)
+    (property "Reference" "#FLG0112" (id 0) (at 143.51 33.655 0)
+      (effects (font (size 1.27 1.27)) hide)
+    )
+    (property "Value" "PWR_FLAG" (id 1) (at 143.51 30.48 0))
+    (property "Footprint" "" (id 2) (at 143.51 35.56 0)
+      (effects (font (size 1.27 1.27)) hide)
+    )
+    (property "Datasheet" "~" (id 3) (at 143.51 35.56 0)
+      (effects (font (size 1.27 1.27)) hide)
+    )
+    (pin "1")
+  )
   (symbol (lib_id "power:+3.3V") (at 109.22 41.91 0) (unit 1)
     (in_bom yes) (on_board yes) (fields_autoplaced)
@@
       (effects (font (size 1.27 1.27)) hide)
     )
+    (pin "1")
+  )
+  (symbol (lib_id "power:PWR_FLAG") (at 130.81 59.69 0) (unit 1)
+    (in_bom yes) (on_board yes) (fields_autoplaced)
+    (property "Reference" "#FLG0104" (id 0) (at 130.81 57.785 0)
+      (effects (font (size 1.27 1.27)) hide)
+    )
+    (property "Value" "PWR_FLAG" (id 1) (at 130.81 54.61 0))
+    (property "Footprint" "" (id 2) (at 130.81 59.69 0)
+      (effects (font (size 1.27 1.27)) hide)
+    )
+    (property "Datasheet" "~" (id 3) (at 130.81 59.69 0)
+      (effects (font (size 1.27 1.27)) hide)
+    )
