File: Strelka_Power_Board/Actuators.kicad_sch (KiCad schematic)
At the start: 29 parts

Commit message: Creating BOM
Parts:
- J? (x4): footprint (none) -> Connector_PinHeader_2.54mm:PinHeader_1x03_P2.54mm_Vertical
- J?: footprint S04BXASK1LFSN -> Footprints:S04BXASK1LFSN; Arrow Part Number S04B-XASK-1(LF)(SN) -> (none); Arrow Price/Stock https://www.arrow.com/en/products/s04b-xask-1-lf-sn/jst-man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 -> (none); Height 7 -> (none); LCSC# (none) -> C265097; Manufacturer_Name JST (JAPAN SOLDERLESS TERMINALS) -> (none); Manufacturer_Part_Number S04B-XASK-1(LF)(SN) -> (none)
Changed lines of the file:
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@@
       (effects (font (size 1.27 1.27)) (justify left))
     )
-    (property "Footprint" "" (id 2) (at 69.342 71.882 0)
+    (property "Footprint" "Connector_PinHeader_2.54mm:PinHeader_1x03_P2.54mm_Vertical" (id 2) (at 69.342 71.882 0)
       (effects (font (size 1.27 1.27)) hide)
     )
@@
       (effects (font (size 1.27 1.27)) (justify left))
     )
-    (property "Footprint" "" (id 2) (at 69.342 59.69 0)
+    (property "Footprint" "Connector_PinHeader_2.54mm:PinHeader_1x03_P2.54mm_Vertical" (id 2) (at 69.342 59.69 0)
       (effects (font (size 1.27 1.27)) hide)
     )
@@
       (effects (font (size 1.27 1.27)) (justify left))
     )
-    (property "Footprint" "" (id 2) (at 69.342 33.02 0)
+    (property "Footprint" "Connector_PinHeader_2.54mm:PinHeader_1x03_P2.54mm_Vertical" (id 2) (at 69.342 33.02 0)
       (effects (font (size 1.27 1.27)) hide)
     )
@@
       (effects (font (size 1.27 1.27)) (justify left))
     )
-    (property "Footprint" "" (id 2) (at 69.342 46.99 0)
+    (property "Footprint" "Connector_PinHeader_2.54mm:PinHeader_1x03_P2.54mm_Vertical" (id 2) (at 69.342 46.99 0)
       (effects (font (size 1.27 1.27)) hide)
     )
@@
     (property "Reference" "J?" (id 0) (at 114.3 125.73 0))
     (property "Value" "S04B-XASK-1_LF__SN_" (id 1) (at 114.3 128.27 0))
-    (property "Footprint" "S04BXASK1LFSN" (id 2) (at 120.65 130.81 0)
+    (property "Footprint" "Footprints:S04BXASK1LFSN" (id 2) (at 120.65 130.81 0)
       (effects (font (size 1.27 1.27)) (justify left) hide)
     )
@@
       (effects (font (size 1.27 1.27)) (justify left) hide)
     )
-    (property "Description" "JST (JAPAN SOLDERLESS TERMINALS) - S04B-XASK-1(LF)(SN) - HEADER, 90DEG, 4WAY" (id 4) (at 120.65 135.89 0)
+    (property "LCSC#" "C265097" (id 4) (at 120.65 135.89 0)
       (effects (font (size 1.27 1.27)) (justify left) hide)
     )
-    (property "Height" "7" (id 5) (at 120.65 138.43 0)
-      (effects (font (size 1.27 1.27)) (justify left) hide)
-    )
-    (property "Manufacturer_Name" "JST (JAPAN SOLDERLESS TERMINALS)" (id 6) (at 120.65 140.97 0)
-      (effects (font (size 1.27 1.27)) (justify left) hide)
-    )
-    (property "Manufacturer_Part_Number" "S04B-XASK-1(LF)(SN)" (id 7) (at 120.65 143.51 0)
-      (effects (font (size 1.27 1.27)) (justify left) hide)
-    )
-    (property "Mouser Part Number" "" (id 8) (at 120.65 146.05 0)
-      (effects (font (size 1.27 1.27)) (justify left) hide)
-    )
-    (property "Mouser Price/Stock" "" (id 9) (at 120.65 148.59 0)
-      (effects (font (size 1.27 1.27)) (justify left) hide)
-    )
-    (property "Arrow Part Number" "S04B-XASK-1(LF)(SN)" (id 10) (at 120.65 151.13 0)
-      (effects (font (size 1.27 1.27)) (justify left) hide)
-    )
-    (property "Arrow Price/Stock" "https://www.arrow.com/en/products/s04b-xask-1-lf-sn/jst-manufacturing" (id 11) (at 120.65 153.67 0)
-      (effects (font (size 1.27 1.27)) (justify left) hide)
-    )
-    (property "Mouser Testing Part Number" "" (id 12) (at 120.65 156.21 0)
-      (effects (font (size 1.27 1.27)) (justify left) hide)
-    )
-    (property "Mouser Testing Price/Stock" "" (id 13) (at 120.65 158.75 0)
-      (effects (font (size 1.27 1.27)) (justify left) hide)
-    )
