File: Strelka_Power_Board/STM32F405.kicad_sch (KiCad schematic)
At the start: 19 parts

Commit message: Creating BOM
Connections:
- net +3V3: now also U?.1 (VBAT)
- no-connect marks 2 -> 1
Other:
- note removed: "CAN WE USE VBAT???"
- moved on the sheet: C?, R?, SW?, U?, Y?
