File: Strelka_Power_Board/Power.kicad_sch (KiCad schematic)
At the start: 9 parts

Commit message: Creating BOM
Parts:
- removed Q?: ??, Package_TO_SOT_SMD:SOT-23, symbol Transistor_FET:Si2319CDS
- added Q?: CJK2333, Package_TO_SOT_SMD:SOT-23, symbol Transistor_FET:Si2319CDS
- SW?: footprint (none) -> Footprints:SM02BGHSTBLFSN
Connections:
- net +BATT: now also Q?.3 (D)
- net at D?.1 (K), SW?.1: now also Q?.2 (S)
- net at D?.2 (A), R?.2: now also Q?.1 (G)
Other:
- moved on the sheet: C?, D?, J?, R?, SW?

Commit message: redo placement
Parts:
- R?: value ? -> 10k; LCSC# C105579 -> (none)
- R?: value ? -> 40k; LCSC# C137796 -> C3016445
Connections:
- net VDC is gone; now on net VCC: R?.2
Other:
- note added: "Vin = 18.6 12.6 8.40 Vo = 3.36 2.52 1.68"
- note removed: "Vin = Vo ="
Changed lines of the file:
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@@
     (stroke (width 0) (type default) (color 0 0 0 0))
   )
-  (text "Vin = \nVo = " (at 120.015 92.075 0)
+  (text "Vin = 18.6 12.6 8.40 \nVo = 3.36 2.52 1.68" (at 120.65 93.345 0)
     (effects (font (size 1.27 1.27)) (justify left bottom))
   )
@@
       (effects (font (size 1.27 1.27)) (justify left))
     )
-    (property "Value" "?" (id 1) (at 115.3414 97.917 0)
+    (property "Value" "10k" (id 1) (at 115.3414 97.917 0)
       (effects (font (size 1.27 1.27)) (justify left))
     )
@@
       (effects (font (size 1.27 1.27)) hide)
     )
-    (property "LCSC#" "C105579" (id 4) (at 116.84 99.06 0)
+    (property "LCSC#" "" (id 4) (at 116.84 99.06 0)
       (effects (font (size 1.27 1.27)) hide)
     )
@@
       (effects (font (size 1.27 1.27)) (justify left))
     )
-    (property "Value" "?" (id 1) (at 115.3414 90.297 0)
+    (property "Value" "40k" (id 1) (at 115.3414 90.297 0)
       (effects (font (size 1.27 1.27)) (justify left))
     )
@@
       (effects (font (size 1.27 1.27)) hide)
     )
-    (property "LCSC#" "C137796" (id 4) (at 116.84 91.44 0)
+    (property "LCSC#" "C3016445" (id 4) (at 116.84 91.44 0)
       (effects (font (size 1.27 1.27)) hide)
     )
@@
     (pin "1")
   )
+  (symbol (lib_id "power:VCC") (at 116.84 88.9 0) (unit 1)
+    (in_bom yes) (on_board yes)
+    (property "Reference" "#PWR?" (id 0) (at 116.84 92.71 0)
+      (effects (font (size 1.27 1.27)) hide)
+    )
+    (property "Value" "VCC" (id 1) (at 118.11 87.63 0)
+      (effects (font (size 1.27 1.27)) (justify left))
+    )
+    (property "Footprint" "" (id 2) (at 116.84 88.9 0)
+      (effects (font (size 1.27 1.27)) hide)
+    )
+    (property "Datasheet" "" (id 3) (at 116.84 88.9 0)
+      (effects (font (size 1.27 1.27)) hide)
+    )
+    (pin "1")
+  )
   (symbol (lib_id "power:-BATT") (at 90.17 73.66 180) (unit 1)
     (in_bom yes) (on_board yes) (fields_autoplaced)
@@
       (effects (font (size 1.27 1.27)) hide)
     )
-    (pin "1")
-  )
-  (symbol (lib_id "power:VDC") (at 116.84 88.9 0) (unit 1)
-    (in_bom yes) (on_board yes) (fields_autoplaced)
-    (property "Reference" "#PWR?" (id 0) (at 116.84 91.44 0)
-      (effects (font (size 1.27 1.27)) hide)
-    )
-    (property "Value" "VDC" (id 1) (at 116.84 84.328 0))
-    (property "Footprint" "" (id 2) (at 116.84 88.9 0)
-      (effects (font (size 1.27 1.27)) hide)
-    )
-    (property "Datasheet" "" (id 3) (at 116.84 88.9 0)
-      (effects (font (size 1.27 1.27)) hide)
-    )
